File: KiCad documents/HybridChargeController.sch (KiCad schematic (older format))
At the start: 90 parts, among them P1 Load, P2 LI_balancer, P3 PV, P4 Extra, P5 LI, P6 LA, Q1 MMBT3904, Q10 MMBT3904, Q11 IPD90P04P4L-04, Q12 STL60P4LLF6, Q13 STL60P4LLF6, Q2 IPD90P04P4L-04, Q3 RQ3E100BNTB, Q4 IPD90P04P4L-04, Q5 RQ3E100BNTB, Q6 MMBT3904, Q7 BSS138, Q8 MMBT3904, Q9 IPD90P04P4L-04, U1 LM358D, U2 bq76920, U3 cd4051, U4 LM358D, U5 LM358D

Commit message: new branch highside switch
Parts:
- removed D1: 1N4148-T, Diodes_ThroughHole:D_DO-35_SOD27_P10.16mm_Horizontal, symbol D
- removed Q3, Q5: RQ3E100BNTB, bachelorSMDs:HSMT-8, symbol RQ3E100BNTB
- removed Q7: BSS138, TO_SOT_Packages_SMD:SOT-23, symbol BSS138
- removed R22, R28, R33: 1M, Resistors_SMD:R_0603_HandSoldering, symbol R
- added Q?: MMBT3904, TO_SOT_Packages_SMD:SOT-23, symbol Q_NPN_BEC
- added Q?: IPD90P04P4L-04, TO_SOT_Packages_SMD:TO-252-3_TabPin2, symbol IPD90P04P4L-04
- added R?: 47k, Resistors_SMD:R_0603_HandSoldering, symbol R
- added R?: 100k, Resistors_SMD:R_0603_HandSoldering, symbol R
- added R?: 10k, Resistors_SMD:R_0603_HandSoldering, symbol R
Connections:
- wire segments 286 -> 266
Changed lines of the file:
@@
 	0    1    1    0
 $EndComp
-$Comp
-L R R22
-U 1 1 58FC76A9
-P 3000 10375
-F 0 "R22" V 3080 10375 50  0000 C CNN
-F 1 "1M" V 3000 10375 50  0000 C CNN
-F 2 "Resistors_SMD:R_0603_HandSoldering" V 2930 10375 50  0001 C CNN
-F 3 "" H 3000 10375 50  0000 C CNN
-	1    3000 10375
-	1    0    0    -1
-$EndComp
-Text Label 3400 10125 0    60   ~ 0
-DSG
 Text Label 2650 7575 2    60   ~ 0
 DSG
-Text Label 5150 10575 0    60   ~ 0
-GND
-$Comp
-L R R33
-U 1 1 58FCBA25
-P 4925 10375
-F 0 "R33" V 5005 10375 50  0000 C CNN
-F 1 "1M" V 4925 10375 50  0000 C CNN
-F 2 "Resistors_SMD:R_0603_HandSoldering" V 4855 10375 50  0001 C CNN
-F 3 "" H 4925 10375 50  0000 C CNN
-	1    4925 10375
-	1    0    0    -1
-$EndComp
-$Comp
-L R R28
-U 1 1 58FCE652
-P 4625 9725
-F 0 "R28" V 4705 9725 50  0000 C CNN
-F 1 "1M" V 4625 9725 50  0000 C CNN
-F 2 "Resistors_SMD:R_0603_HandSoldering" V 4555 9725 50  0001 C CNN
-F 3 "" H 4625 9725 50  0000 C CNN
-	1    4625 9725
-	1    0    0    -1
-$EndComp
-$Comp
-L D D1
-U 1 1 58FCE732
-P 4925 9725
-F 0 "D1" H 4925 9825 50  0000 C CNN
-F 1 "1N4148-T" H 4925 9625 50  0000 C CNN
-F 2 "Diodes_ThroughHole:D_DO-35_SOD27_P10.16mm_Horizontal" H 4925 9725 50  0001 C CNN
-F 3 "" H 4925 9725 50  0000 C CNN
-	1    4925 9725
-	0    -1   -1   0
-$EndComp
-Text Label 4175 9225 0    60   ~ 0
-GND
-Text Label 4725 8825 0    60   ~ 0
-CHG
 Text Label 2650 7675 2    60   ~ 0
 CHG
@@
 	2400 1450 2850 1450
 Wire Wire Line
-	5700 5000 5700 5000
+	5700 5000 6100 5000
+Wire Wire Line
+	6100 5000 6600 5000
 Connection ~ 6100 5000
 Wire Wire Line
@@
 Wire Wire Line
 	6100 5000 6100 5100
-Wire Wire Line
-	5700 5000 6100 5000
-Wire Wire Line
-	6100 5000 6600 5000
 Wire Wire Line
 	800  8975 1150 8975
@@
 	2650 10625 2700 10625
 Wire Wire Line
-	2700 10625 3000 10625
-Wire Wire Line
-	3000 10625 3100 10625
-Wire Wire Line
-	3100 10625 3175 10625
-Wire Wire Line
-	3175 10625 3250 10625
-Wire Wire Line
-	3000 10525 3000 10625
-Connection ~ 3000 10625
-Wire Wire Line
-	3000 10225 3400 10225
-Wire Wire Line
-	3400 10125 3400 10225
-Wire Wire Line
-	3400 10225 3400 10450
-Connection ~ 3400 10225
-Wire Wire Line
-	4625 10175 4625 10450
-Wire Wire Line
-	4925 9875 4925 9975
-Wire Wire Line
-	4925 9975 4925 10175
-Wire Wire Line
-	4925 10175 4925 10225
-Connection ~ 4925 10175
-Wire Wire Line
-	4625 9875 4625 9975
-Wire Wire Line
-	4625 9975 4925 9975
-Connection ~ 4925 9975
-Wire Wire Line
-	4425 9225 4175 9225
-Wire Wire Line
-	4925 9475 4925 9575
-Wire Wire Line
-	4625 9475 4725 9475
-Wire Wire Line
-	4725 9475 4925 9475
-Wire Wire Line
-	4625 9475 4625 9575
-Wire Wire Line
-	4725 9375 4725 9475
-Connection ~ 4725 9475
-Wire Wire Line
-	4725 8975 4725 8825
+	2700 10625 4600 10625
+Wire Wire Line
+	4600 10625 5075 10625
+Wire Wire Line
+	5075 10625 5700 10625
 Wire Wire Line
 	2650 8175 2150 8175
@@
 Connection ~ 2300 10625
 Wire Wire Line
-	2700 10475 2700 10625
+	2700 10625 2700 10475
 Connection ~ 2700 10625
 Wire Wire Line
@@
 	650  7175 650  11200
 Wire Notes Line
-	650  7175 5550 7175
-Wire Notes Line
-	5550 7175 5550 11200
-Wire Notes Line
-	5550 11200 650  11200
+	650  7175 6625 7175
+Wire Notes Line
+	6625 7175 6625 11200
+Wire Notes Line
+	6625 11200 650  11200
 Wire Wire Line
 	7000 3350 6950 3350
@@
 Text Label 8750 6900 1    60   ~ 0
 D9
-Wire Wire Line
-	4925 10175 4625 10175
-$Comp
-L BSS138 Q7
-U 1 1 5905B77E
-P 4625 9175
-F 0 "Q7" H 4825 9250 50  0000 L CNN
-F 1 "BSS138" H 4825 9175 50  0000 L CNN
-F 2 "TO_SOT_Packages_SMD:SOT-23" H 4825 9100 50  0001 L CIN
-F 3 "" H 4625 9175 50  0000 L CNN
-	1    4625 9175
-	1    0    0    -1
-$EndComp
 $Comp
 L R R3
@@
 short!
 $Comp
-L RQ3E100BNTB Q3
-U 1 1 59128DBA
-P 3500 10825
-F 0 "Q3" V 3200 10875 60  0000 C CNN
-F 1 "RQ3E100BNTB" V 3775 10825 60  0000 C CNN
-F 2 "bachelorSMDs:HSMT-8" H 3500 10825 60  0001 C CNN
-F 3 "" H 3500 10825 60  0001 C CNN
-	1    3500 10825
-	0    1    1    0
-$EndComp
-Connection ~ 3100 10625
-Connection ~ 3175 10625
-Wire Wire Line
-	3725 10625 3800 10625
-Wire Wire Line
-	3800 10625 3875 10625
-Wire Wire Line
-	3875 10625 3950 10625
-Wire Wire Line
-	3950 10625 4075 10625
-Wire Wire Line
-	4075 10625 4150 10625
-Wire Wire Line
-	4150 10625 4225 10625
-Wire Wire Line
-	4225 10625 4300 10625
-Connection ~ 3800 10625
-Connection ~ 3875 10625
-$Comp
-L RQ3E100BNTB Q5
-U 1 1 5912D7B6
-P 4525 10825
-F 0 "Q5" V 4225 10875 60  0000 C CNN
-F 1 "RQ3E100BNTB" V 4775 10825 60  0000 C CNN
-F 2 "bachelorSMDs:HSMT-8" H 4525 10825 60  0001 C CNN
-F 3 "" H 4525 10825 60  0001 C CNN
-	1    4525 10825
-	0    -1   1    0
-$EndComp
-Connection ~ 3950 10625
-Connection ~ 4075 10625
-Connection ~ 4150 10625
-Connection ~ 4225 10625
-Wire Wire Line
-	4925 10625 4850 10625
-Wire Wire Line
-	4850 10625 4775 10625
-Connection ~ 4850 10625
-Wire Wire Line
-	4925 10525 4925 10575
-Wire Wire Line
-	4925 10575 4925 10625
-Wire Wire Line
-	4925 10575 5150 10575
-Connection ~ 4925 10575
-$Comp
 L Q_NPN_BEC Q1
 U 1 1 59149D07
@@
 	0    1    1    0
 $EndComp
+$Comp
+L R R?
+U 1 1 591B35A8
+P 4775 9725
+F 0 "R?" V 4855 9725 50  0000 C CNN
+F 1 "47k" V 4775 9725 50  0000 C CNN
+F 2 "Resistors_SMD:R_0603_HandSoldering" V 4705 9725 50  0001 C CNN
+F 3 "" H 4775 9725 50  0000 C CNN
+	1    4775 9725
+	0    1    1    0
+$EndComp
+$Comp
+L R R?
+U 1 1 591B35AE
+P 4600 10275
+F 0 "R?" V 4680 10275 50  0000 C CNN
+F 1 "100k" V 4600 10275 50  0000 C CNN
+F 2 "Resistors_SMD:R_0603_HandSoldering" V 4530 10275 50  0001 C CNN
+F 3 "" H 4600 10275 50  0000 C CNN
+	1    4600 10275
+	-1   0    0    1
+$EndComp
+Text Label 4175 10025 2    60   ~ 0
+SW_LD
+Text Label 5700 9425 0    60   ~ 0
+COM+
+$Comp
+L R R?
+U 1 1 591B35B7
+P 4325 10025
+F 0 "R?" V 4405 10025 50  0000 C CNN
+F 1 "10k" V 4325 10025 50  0000 C CNN
+F 2 "Resistors_SMD:R_0603_HandSoldering" V 4255 10025 50  0001 C CNN
+F 3 "" H 4325 10025 50  0000 C CNN
+	1    4325 10025
+	0    1    1    0
+$EndComp
+Wire Wire Line
+	5075 9725 5075 9825
+Connection ~ 5075 9725
+Wire Wire Line
+	4350 9425 4625 9425
+Wire Wire Line
+	4625 9425 4925 9425
+Connection ~ 4625 9425
+Wire Wire Line
+	4625 9725 4625 9425
+Connection ~ 4600 10025
+Wire Wire Line
+	4600 10025 4600 10125
+Wire Wire Line
+	4475 10025 4600 10025
+Wire Wire Line
+	4600 10025 4775 10025
+Connection ~ 4600 10625
+Wire Wire Line
+	4600 10625 4600 10425
+Connection ~ 5075 10625
+Wire Wire Line
+	5075 10625 5075 10225
+Wire Wire Line
+	4925 9725 5075 9725
+Wire Wire Line
+	5075 9725 5175 9725
+$Comp
+L Q_NPN_BEC Q?
+U 1 1 591B35CC
+P 4975 10025
+F 0 "Q?" H 5275 10075 50  0000 R CNN
+F 1 "MMBT3904" H 5575 9975 50  0000 R CNN
+F 2 "TO_SOT_Packages_SMD:SOT-23" H 5175 10125 50  0001 C CNN
+F 3 "" H 4975 10025 50  0000 C CNN
+	1    4975 10025
+	1    0    0    -1
+$EndComp
+$Comp
+L IPD90P04P4L-04 Q?
+U 1 1 591B35D2
+P 5275 9425
+F 0 "Q?" V 5400 9125 60  0000 C CNN
+F 1 "IPD90P04P4L-04" V 5525 9475 60  0000 C CNN
+F 2 "TO_SOT_Packages_SMD:TO-252-3_TabPin2" H 5275 9425 60  0001 C CNN
+F 3 "" H 5275 9425 60  0001 C CNN
+	1    5275 9425
+	0    -1   -1   0
+$EndComp
+Wire Wire Line
+	5700 9425 5600 9425
+Text Label 5700 10625 0    60   ~ 0
+GND
 $EndSCHEMATC

Commit message: implemented new HS switch
Parts:
- added Q?: IPD90P04P4L-04, TO_SOT_Packages_SMD:TO-252-3_TabPin2, symbol IPD90P04P4L-04
- added Q?: MMBT3904, TO_SOT_Packages_SMD:SOT-23, symbol Q_NPN_BEC
- added R?: 47k, Resistors_SMD:R_0603_HandSoldering, symbol R
- added R?: 100k, Resistors_SMD:R_0603_HandSoldering, symbol R
- added R?: 10k, Resistors_SMD:R_0603_HandSoldering, symbol R
Connections:
- wire segments 266 -> 192
Other:
- moved on the sheet: Q?, R?

Commit message: startet distributing components
Parts:
- gave numbers to parts that had none: 10
Changed lines of the file:
@@
 $EndComp
 $Comp
-L R R?
+L R R52
 U 1 1 591B35A8
 P 5400 9725
-F 0 "R?" V 5480 9725 50  0000 C CNN
+F 0 "R52" V 5480 9725 50  0000 C CNN
 F 1 "47k" V 5400 9725 50  0000 C CNN
 F 2 "Resistors_SMD:R_0603_HandSoldering" V 5330 9725 50  0001 C CNN
@@
 $EndComp
 $Comp
-L R R?
+L R R51
 U 1 1 591B35AE
 P 5225 10275
-F 0 "R?" V 5305 10275 50  0000 C CNN
+F 0 "R51" V 5305 10275 50  0000 C CNN
 F 1 "100k" V 5225 10275 50  0000 C CNN
 F 2 "Resistors_SMD:R_0603_HandSoldering" V 5155 10275 50  0001 C CNN
@@
 COM+
 $Comp
-L R R?
+L R R33
 U 1 1 591B35B7
 P 4950 10025
-F 0 "R?" V 5030 10025 50  0000 C CNN
+F 0 "R33" V 5030 10025 50  0000 C CNN
 F 1 "10k" V 4950 10025 50  0000 C CNN
 F 2 "Resistors_SMD:R_0603_HandSoldering" V 4880 10025 50  0001 C CNN
@@
 $EndComp
 $Comp
-L Q_NPN_BEC Q?
+L Q_NPN_BEC Q7
 U 1 1 591B35CC
 P 5600 10025
-F 0 "Q?" H 5900 10075 50  0000 R CNN
+F 0 "Q7" H 5900 10075 50  0000 R CNN
 F 1 "MMBT3904" H 6200 9975 50  0000 R CNN
 F 2 "TO_SOT_Packages_SMD:SOT-23" H 5800 10125 50  0001 C CNN
@@
 $EndComp
 $Comp
-L IPD90P04P4L-04 Q?
+L IPD90P04P4L-04 Q14
 U 1 1 591B35D2
 P 5900 9425
-F 0 "Q?" V 6025 9125 60  0000 C CNN
+F 0 "Q14" V 6025 9125 60  0000 C CNN
 F 1 "IPD90P04P4L-04" V 6150 9475 60  0000 C CNN
 F 2 "TO_SOT_Packages_SMD:TO-252-3_TabPin2" H 5900 9425 60  0001 C CNN
@@
 GND
 $Comp
-L IPD90P04P4L-04 Q?
+L IPD90P04P4L-04 Q5
 U 1 1 591C2F97
 P 4750 9425
-F 0 "Q?" V 4875 9125 60  0000 C CNN
+F 0 "Q5" V 4875 9125 60  0000 C CNN
 F 1 "IPD90P04P4L-04" V 5000 9475 60  0000 C CNN
 F 2 "TO_SOT_Packages_SMD:TO-252-3_TabPin2" H 4750 9425 60  0001 C CNN
@@
 $EndComp
 $Comp
-L R R?
+L R R50
 U 1 1 591C3122
 P 5075 9000
-F 0 "R?" V 5155 9000 50  0000 C CNN
+F 0 "R50" V 5155 9000 50  0000 C CNN
 F 1 "47k" V 5075 9000 50  0000 C CNN
 F 2 "Resistors_SMD:R_0603_HandSoldering" V 5005 9000 50  0001 C CNN
@@
 	5225 9000 5250 9000
 $Comp
-L Q_NPN_BEC Q?
+L Q_NPN_BEC Q3
 U 1 1 591C41F7
 P 4100 10025
-F 0 "Q?" H 4400 10075 50  0000 R CNN
+F 0 "Q3" H 4400 10075 50  0000 R CNN
 F 1 "MMBT3904" H 4700 9975 50  0000 R CNN
 F 2 "TO_SOT_Packages_SMD:SOT-23" H 4300 10125 50  0001 C CNN
@@
 Connection ~ 4850 9000
 $Comp
-L R R?
+L R R28
 U 1 1 591C5F0A
 P 3800 10275
-F 0 "R?" V 3880 10275 50  0000 C CNN
+F 0 "R28" V 3880 10275 50  0000 C CNN
 F 1 "100k" V 3800 10275 50  0000 C CNN
 F 2 "Resistors_SMD:R_0603_HandSoldering" V 3730 10275 50  0001 C CNN
@@
 CHG
 $Comp
-L R R?
+L R R22
 U 1 1 591C5F11
 P 3525 10025
-F 0 "R?" V 3605 10025 50  0000 C CNN
+F 0 "R22" V 3605 10025 50  0000 C CNN
 F 1 "10k" V 3525 10025 50  0000 C CNN
 F 2 "Resistors_SMD:R_0603_HandSoldering" V 3455 10025 50  0001 C CNN

Commit message: completed vaguely arranging footprints
Other:
- moved on the sheet: D3, R38, R39, R41, R42
Changed lines of the file:
@@
 	0    1    1    0
 $EndComp
-Text Label 7200 2350 2    60   ~ 0
+Text Label 6750 2350 2    60   ~ 0
 PV-
-Text Label 9950 1750 0    60   ~ 0
+Text Label 6875 1775 2    60   ~ 0
 S_PV_V
 $Comp
@@
 L R R42
 U 1 1 58F03300
-P 9800 2000
-F 0 "R42" V 9880 2000 50  0000 C CNN
-F 1 "33k" V 9800 2000 50  0000 C CNN
-F 2 "Resistors_SMD:R_0603_HandSoldering" V 9730 2000 50  0001 C CNN
-F 3 "" H 9800 2000 50  0000 C CNN
-	1    9800 2000
+P 6950 2025
+F 0 "R42" V 7030 2025 50  0000 C CNN
+F 1 "33k" V 6950 2025 50  0000 C CNN
+F 2 "Resistors_SMD:R_0603_HandSoldering" V 6880 2025 50  0001 C CNN
+F 3 "" H 6950 2025 50  0000 C CNN
+	1    6950 2025
 	1    0    0    -1
 $EndComp
@@
 L R R41
 U 1 1 58F03306
-P 9800 1500
-F 0 "R41" V 9880 1500 50  0000 C CNN
-F 1 "100k" V 9800 1500 50  0000 C CNN
-F 2 "Resistors_SMD:R_0603_HandSoldering" V 9730 1500 50  0001 C CNN
-F 3 "" H 9800 1500 50  0000 C CNN
-	1    9800 1500
+P 6950 1525
+F 0 "R41" V 7030 1525 50  0000 C CNN
+F 1 "100k" V 6950 1525 50  0000 C CNN
+F 2 "Resistors_SMD:R_0603_HandSoldering" V 6880 1525 50  0001 C CNN
+F 3 "" H 6950 1525 50  0000 C CNN
+	1    6950 1525
 	1    0    0    -1
 $EndComp
@@
 	0    1    1    0
 $EndComp
-Text Label 9600 1150 2    60   ~ 0
-PV+
 Text Label 11700 1150 0    60   ~ 0
 COM+
@@
 	0    -1   -1   0
 $EndComp
+Text Label 10075 7500 3    60   ~ 0
+LOAD-
 Text Label 10175 7500 3    60   ~ 0
-LOAD-
-Text Label 10075 7500 3    60   ~ 0
 LOAD+
-Text Label 10725 7500 3    60   ~ 0
+Text Label 10625 7500 3    60   ~ 0
 PV-
 Text Label 12225 9000 3    60   ~ 0
 LA-
-Text Label 10625 8100 3    60   ~ 0
+Text Label 10725 8100 3    60   ~ 0
 PV+
 Text Label 12425 9000 3    60   ~ 0
@@
 L D D3
 U 1 1 58F0B98B
-P 10625 7950
-F 0 "D3" H 10625 8050 50  0000 C CNN
-F 1 "VSB2045Y-M3/54" H 10625 7850 50  0000 C CNN
-F 2 "Diodes_ThroughHole:D_P600_R-6_P12.70mm_Horizontal" H 10625 7950 50  0001 C CNN
-F 3 "" H 10625 7950 50  0000 C CNN
-	1    10625 7950
+P 10725 7950
+F 0 "D3" H 10725 8050 50  0000 C CNN
+F 1 "VSB2045Y-M3/54" H 10725 7850 50  0000 C CNN
+F 2 "Diodes_ThroughHole:D_P600_R-6_P12.70mm_Horizontal" H 10725 7950 50  0001 C CNN
+F 3 "" H 10725 7950 50  0000 C CNN
+	1    10725 7950
 	0    -1   -1   0
 $EndComp
@@
 L R R39
 U 1 1 58EE841A
-P 7500 2000
-F 0 "R39" V 7580 2000 50  0000 C CNN
-F 1 "100k" V 7500 2000 50  0000 C CNN
-F 2 "Resistors_SMD:R_0603_HandSoldering" V 7430 2000 50  0001 C CNN
-F 3 "" H 7500 2000 50  0000 C CNN
-	1    7500 2000
+P 7950 2000
+F 0 "R39" V 8030 2000 50  0000 C CNN
+F 1 "100k" V 7950 2000 50  0000 C CNN
+F 2 "Resistors_SMD:R_0603_HandSoldering" V 7880 2000 50  0001 C CNN
+F 3 "" H 7950 2000 50  0000 C CNN
+	1    7950 2000
 	-1   0    0    1
 $EndComp
-Text Label 7000 1750 2    60   ~ 0
+Text Label 7600 1750 2    60   ~ 0
 SW_PV
 Text Notes 6500 800  0    60   ~ 0
@@
 L R R38
 U 1 1 58EE8440
-P 7150 1750
-F 0 "R38" V 7230 1750 50  0000 C CNN
-F 1 "10k" V 7150 1750 50  0000 C CNN
-F 2 "Resistors_SMD:R_0603_HandSoldering" V 7080 1750 50  0001 C CNN
-F 3 "" H 7150 1750 50  0000 C CNN
-	1    7150 1750
-	0    1    1    0
-$EndComp
-Text Label 7150 1150 2    60   ~ 0
+P 7750 1750
+F 0 "R38" V 7830 1750 50  0000 C CNN
+F 1 "10k" V 7750 1750 50  0000 C CNN
+F 2 "Resistors_SMD:R_0603_HandSoldering" V 7680 1750 50  0001 C CNN
+F 3 "" H 7750 1750 50  0000 C CNN
+	1    7750 1750
+	0    1    1    0
+$EndComp
+Text Label 6750 1150 2    60   ~ 0
 PV+
 Text Notes 9675 10825 0    139  ~ 28
@@
 NoConn ~ 7000 3150
 Text Label 8850 6900 1    60   ~ 0
-D8
+SW_PV
 Text Label 8750 6900 1    60   ~ 0
 D9
@@
 $EndComp
 Wire Wire Line
-	7150 1150 8300 1150
+	6750 1150 8300 1150
 Connection ~ 7850 1150
 Wire Wire Line
@@
 Wire Notes Line
 	6450 2500 6450 600
-Connection ~ 7500 1750
-Wire Wire Line
-	7500 1750 7500 1850
-Wire Wire Line
-	7300 1750 8000 1750
-Connection ~ 7500 2350
-Wire Wire Line
-	7500 2150 7500 2350
+Connection ~ 7950 1750
+Wire Wire Line
+	7950 1750 7950 1850
+Wire Wire Line
+	7900 1750 8000 1750
+Connection ~ 7950 2350
+Wire Wire Line
+	7950 2350 7950 2150
 Connection ~ 8300 2350
 Wire Wire Line
@@
 	9400 600  12050 600
 Wire Wire Line
-	10625 7500 10625 7800
+	10725 7500 10725 7800
 Wire Wire Line
 	12375 7600 12525 7600
@@
 	10300 2350 10300 1350
 Wire Wire Line
-	7200 2350 10300 2350
-Connection ~ 9800 1750
-Wire Wire Line
-	9950 1750 9800 1750
-Connection ~ 9800 2350
-Wire Wire Line
-	9800 2150 9800 2350
-Wire Wire Line
-	9800 1650 9800 1850
-Connection ~ 9800 1150
-Wire Wire Line
-	9800 1150 9800 1350
+	6750 2350 10300 2350
+Connection ~ 6950 1775
+Wire Wire Line
+	6875 1775 6950 1775
+Wire Wire Line
+	6950 1675 6950 1875
+Wire Wire Line
+	6950 1150 6950 1375
 Connection ~ 9100 8900
 Wire Wire Line
@@
 Text Label 1850 8300 2    60   ~ 0
 5V
+Connection ~ 6950 1150
+Wire Wire Line
+	6950 2175 6950 2350
+Connection ~ 6950 2350
 $EndSCHEMATC

Commit message: power paths done
Parts:
- added Q15, Q16: BSS138, TO_SOT_Packages_SMD:SOT-23, symbol BSS138
- added R53, R54, R55, R56: 10k, Resistors_SMD:R_0603_HandSoldering, symbol R
- AU1: footprint Arduinos:ARDUINO_SHIELD_bigger_holes -> Arduinos:ARDUINO_SHIELD_bigger_holes_no_outline
- P4: footprint Pin_Headers:Pin_Header_Straight_1x07_Pitch2.54mm -> Pin_Headers:Pin_Header_Straight_1x06_Pitch2.54mm; symbol CONN_01X07 -> CONN_01X06
Connections:
- net labels added: 3.3V, SCL3, SCL5, SDA3, SDA5
- net labels removed: D5, D8, SCL, SDA
- wire segments 192 -> 210
Other:
- note added: "Levelshifter"
Changed lines of the file:
@@
 F 0 "AU1" H 8050 7750 60  0000 C CNN
 F 1 "Uno Layout" H 8800 7550 60  0000 C CNN
-F 2 "Arduinos:ARDUINO_SHIELD_bigger_holes" H 7350 7600 60  0001 C CNN
+F 2 "Arduinos:ARDUINO_SHIELD_bigger_holes_no_outline" H 7350 7600 60  0001 C CNN
 F 3 "" H 7350 7600 60  0001 C CNN
 	1    7350 7600
@@
 Alert
 Text Label 2650 7875 2    60   ~ 0
-SDA
+SDA3
 Text Label 2650 7975 2    60   ~ 0
-SCL
+SCL3
 Text Label 9350 8450 3    60   ~ 0
-SDA
+SDA5
 Text Label 9250 8450 3    60   ~ 0
-SCL
+SCL5
 $Comp
 L R R16
@@
 15A max current measuring
 NoConn ~ 8150 6900
-Text Label 10975 6825 3    60   ~ 0
+Text Label 10925 6825 3    60   ~ 0
 D9
 $Comp
-L CONN_01X07 P4
+L CONN_01X06 P4
 U 1 1 5904BFED
 P 10775 6625
 F 0 "P4" H 10775 7025 50  0000 C CNN
 F 1 "Extra" V 10875 6625 50  0000 C CNN
-F 2 "Pin_Headers:Pin_Header_Straight_1x07_Pitch2.54mm" H 10775 6625 50  0001 C CNN
+F 2 "Pin_Headers:Pin_Header_Straight_1x06_Pitch2.54mm" H 10775 6625 50  0001 C CNN
 F 3 "" H 10775 6625 50  0000 C CNN
 	1    10775 6625
 	0    -1   -1   0
 $EndComp
-Text Label 10475 6825 3    60   ~ 0
+Text Label 10525 6825 3    60   ~ 0
 SCK
-Text Label 10575 6825 3    60   ~ 0
+Text Label 10625 6825 3    60   ~ 0
 MISO
-Text Label 10675 6825 3    60   ~ 0
+Text Label 10725 6825 3    60   ~ 0
 MOSI
-Text Label 10775 6825 3    60   ~ 0
-D5
-Text Label 10875 6825 3    60   ~ 0
-D8
-Text Label 11075 6825 3    60   ~ 0
+Text Label 10825 6825 3    60   ~ 0
+LED_BTN
+Text Label 11025 6825 3    60   ~ 0
 RST
 NoConn ~ 7000 2950
@@
 	6950 2175 6950 2350
 Connection ~ 6950 2350
+$Comp
+L BSS138 Q15
+U 1 1 591C6530
+P 9575 4975
+F 0 "Q15" H 9775 5050 50  0000 L CNN
+F 1 "BSS138" H 9775 4975 50  0000 L CNN
+F 2 "TO_SOT_Packages_SMD:SOT-23" H 9775 4900 50  0001 L CIN
+F 3 "" H 9575 4975 50  0000 L CNN
+	1    9575 4975
+	0    1    1    0
+$EndComp
+$Comp
+L R R53
+U 1 1 591C6613
+P 9250 4725
+F 0 "R53" V 9330 4725 50  0000 C CNN
+F 1 "10k" V 9250 4725 50  0000 C CNN
+F 2 "Resistors_SMD:R_0603_HandSoldering" V 9180 4725 50  0001 C CNN
+F 3 "" H 9250 4725 50  0000 C CNN
+	1    9250 4725
+	1    0    0    -1
+$EndComp
+$Comp
+L R R54
+U 1 1 591C6771
+P 9825 4725
+F 0 "R54" V 9905 4725 50  0000 C CNN
+F 1 "10k" V 9825 4725 50  0000 C CNN
+F 2 "Resistors_SMD:R_0603_HandSoldering" V 9755 4725 50  0001 C CNN
+F 3 "" H 9825 4725 50  0000 C CNN
+	1    9825 4725
+	1    0    0    -1
+$EndComp
+Wire Wire Line
+	9525 4425 9525 4775
+Wire Wire Line
+	8900 4425 9525 4425
+Wire Wire Line
+	9250 4425 9250 4575
+Connection ~ 9250 4425
+Text Label 8900 4425 2    60   ~ 0
+3.3V
+Wire Wire Line
+	9825 4575 9825 4425
+Wire Wire Line
+	9825 4425 9950 4425
+Text Label 9950 4425 0    60   ~ 0
+5V
+Wire Wire Line
+	9250 4875 9250 5500
+Wire Wire Line
+	9375 5075 9250 5075
+Connection ~ 9250 5075
+Wire Wire Line
+	9775 5075 9825 5075
+Wire Wire Line
+	9825 4875 9825 5500
+Connection ~ 9825 5075
+Text Label 9250 5500 3    60   ~ 0
+SDA3
+Text Label 9825 5500 3    60   ~ 0
+SDA5
+Text Label 8650 8450 3    60   ~ 0
+3.3V
+$Comp
+L BSS138 Q16
+U 1 1 591CB903
+P 11075 4975
+F 0 "Q16" H 11275 5050 50  0000 L CNN
+F 1 "BSS138" H 11275 4975 50  0000 L CNN
+F 2 "TO_SOT_Packages_SMD:SOT-23" H 11275 4900 50  0001 L CIN
+F 3 "" H 11075 4975 50  0000 L CNN
+	1    11075 4975
+	0    1    1    0
+$EndComp
+$Comp
+L R R55
+U 1 1 591CB909
+P 10750 4725
+F 0 "R55" V 10830 4725 50  0000 C CNN
+F 1 "10k" V 10750 4725 50  0000 C CNN
+F 2 "Resistors_SMD:R_0603_HandSoldering" V 10680 4725 50  0001 C CNN
+F 3 "" H 10750 4725 50  0000 C CNN
+	1    10750 4725
+	1    0    0    -1
+$EndComp
+$Comp
+L R R56
+U 1 1 591CB90F
+P 11325 4725
+F 0 "R56" V 11405 4725 50  0000 C CNN
+F 1 "10k" V 11325 4725 50  0000 C CNN
+F 2 "Resistors_SMD:R_0603_HandSoldering" V 11255 4725 50  0001 C CNN
+F 3 "" H 11325 4725 50  0000 C CNN
+	1    11325 4725
+	1    0    0    -1
+$EndComp
+Wire Wire Line
+	11025 4425 11025 4775
+Wire Wire Line
+	10400 4425 11025 4425
+Wire Wire Line
+	10750 4425 10750 4575
+Connection ~ 10750 4425
+Text Label 10400 4425 2    60   ~ 0
+3.3V
+Wire Wire Line
+	11325 4575 11325 4425
+Wire Wire Line
+	11325 4425 11450 4425
+Text Label 11450 4425 0    60   ~ 0
+5V
+Wire Wire Line
+	10750 4875 10750 5500
+Wire Wire Line
+	10875 5075 10750 5075
+Connection ~ 10750 5075
+Wire Wire Line
+	11275 5075 11325 5075
+Wire Wire Line
+	11325 4875 11325 5500
+Connection ~ 11325 5075
+Text Label 10750 5500 3    60   ~ 0
+SCL3
+Text Label 11325 5500 3    60   ~ 0
+SCL5
+Text Notes 8700 4200 0    60   ~ 0
+Levelshifter
+Wire Notes Line
+	8650 4100 8650 5900
+Wire Notes Line
+	8650 5900 11675 5900
+Wire Notes Line
+	11675 5900 11675 4100
+Wire Notes Line
+	11675 4100 8650 4100
 $EndSCHEMATC

Commit message: more traces done
Parts:
- P4: footprint Pin_Headers:Pin_Header_Straight_1x06_Pitch2.54mm -> Pin_Headers:Pin_Header_Straight_1x05_Pitch2.54mm; symbol CONN_01X06 -> CONN_01X05
Connections:
- net Alert: now also AU1.9 (D9)
- net RST: now also P4.5 (P5); no longer P4.6 (P6)
- removed net D9: AU1.9 (D9), P4.5 (P5)
Changed lines of the file:
@@
 15A max current measuring
 NoConn ~ 8150 6900
-Text Label 10925 6825 3    60   ~ 0
-D9
 $Comp
-L CONN_01X06 P4
+L CONN_01X05 P4
 U 1 1 5904BFED
 P 10775 6625
 F 0 "P4" H 10775 7025 50  0000 C CNN
 F 1 "Extra" V 10875 6625 50  0000 C CNN
-F 2 "Pin_Headers:Pin_Header_Straight_1x06_Pitch2.54mm" H 10775 6625 50  0001 C CNN
+F 2 "Pin_Headers:Pin_Header_Straight_1x05_Pitch2.54mm" H 10775 6625 50  0001 C CNN
 F 3 "" H 10775 6625 50  0000 C CNN
 	1    10775 6625
 	0    -1   -1   0
 $EndComp
-Text Label 10525 6825 3    60   ~ 0
+Text Label 10575 6825 3    60   ~ 0
 SCK
-Text Label 10625 6825 3    60   ~ 0
+Text Label 10675 6825 3    60   ~ 0
 MISO
-Text Label 10725 6825 3    60   ~ 0
+Text Label 10775 6825 3    60   ~ 0
 MOSI
-Text Label 10825 6825 3    60   ~ 0
+Text Label 10875 6825 3    60   ~ 0
 LED_BTN
-Text Label 11025 6825 3    60   ~ 0
+Text Label 10975 6825 3    60   ~ 0
 RST
 NoConn ~ 7000 2950
@@
 SW_PV
 Text Label 8750 6900 1    60   ~ 0
-D9
+Alert
 $Comp
 L R R3
